File: VFDDriver.kicad_sch (KiCad schematic)
At the start: 30 parts

Commit message: Added input protection components.
Parts:
- added D? (x4): 3V3, symbol Device:D_Zener
- added R? (x4): 200R, symbol Device:R
- added R? (x2): 10R, symbol Device:R
Connections:
- net GND: now also D?.2 (A), D?.2 (A), D?.2 (A), D?.2 (A)
- net VHG: now also R?.2; no longer C?.1, D?.1 (K), D?.2 (A)
- net VHP: now also R?.2; no longer C?.1, D?.1 (K)
- new net: C?.1, D?.1 (K), R?.1
- new net: C?.1, D?.1 (K), D?.2 (A), R?.1
- new net: D?.1 (K), R?.2 (x4)
Other:
- moved on the sheet: C?, D?, L?, R?, U?
